File: hardware/electronics/ControlBoard/Hackerboat Control Board.brd (EAGLE design)
At the start: 114.3 x 195.6 mm, 287 parts, among them IC1 74AHC1G08DBV, IC2 74AUC1G06DBV, IC3 74AHC1G04DBV, IC4 V7805, IC5 7805TV, T1 AO4407A, U1 IPS6041G, U10 INA169, U11 IPS6041G, U12 INA169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

Commit message: More fiddling around with the silkscreen
Parts:
- removed U$6: RS485SOIC, SparkFun-DigitalIC:SO08
- added U28: RS485SOIC, SparkFun-DigitalIC:SO08
- moved C20 190.9 mm to (100.3, 113.0), turned to 270 degrees
- moved C19 177.3 mm to (85.1, 113.0), turned to 270 degrees
- moved F2 166.4 mm to (103.5, 76.2), flipped to the bottom, turned to 180 degrees
- moved IC5 165.2 mm to (92.7, 115.6)
- moved C47 8.28 mm to (77.5, 57.8)
- moved J2 8.28 mm to (84.5, 78.7)
- moved BBB_RESET 8.28 mm to (87.6, 61.0)
- moved D25 8.28 mm to (79.4, 41.3)
- moved D26 8.28 mm to (79.4, 47.6)
- moved D28 8.28 mm to (77.5, 55.9)
- moved IC3 8.28 mm to (77.5, 61.0)
- moved J3 8.28 mm to (84.5, 48.3)
- moved R93 8.28 mm to (79.4, 45.7)
- moved R94 8.28 mm to (79.4, 43.2)
- moved R96 8.28 mm to (81.3, 61.0)
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- renumbered J4 to ENABLE/DISARM
Connections:
- net +5V: now also U28.8; no longer U$6.8
- net BBB_UART1_RX_5V: now also U28.1; no longer U$6.1
- net BBB_UART1_TX_5V: now also U28.4; no longer U$6.4
- net GND: now also U28.5; no longer U$6.5
- net N$27: now also U28.7; no longer U$6.7
- net N$86: now also U28.6; no longer U$6.6
- net RS_485_DIR_SELECT_5V: now also U28.2, U28.3; no longer U$6.2, U$6.3
Routing:
- net N$68: track 0.00 -> 51.0 mm, vias 0 -> 2
- net +12V: track 310.6 -> 343.2 mm
- net +5V: track 882.6 -> 899.1 mm, vias 47 -> 48
- net N$62: track 3.05 -> 16.7 mm, vias 0 -> 1
- net +7V4: track 133.5 -> 142.4 mm
- net BBB_UART0_TX: track 35.7 -> 26.8 mm
- net BBB_UART0_RX: track 35.7 -> 26.8 mm
- net RS_485_DIR_SELECT_5V: track 117.6 -> 126.1 mm
- net BBB_RESET_5V: track 76.0 -> 84.5 mm
- net BBB_STATUS_LIGHTS_5V: track 58.0 -> 66.5 mm
- net BBB_UART1_RX_5V: track 58.6 -> 66.5 mm
- net SERVO_RUDDER_5V: track 42.9 -> 50.9 mm
- net BBB_UART1_TX_5V: track 71.5 -> 79.4 mm
- net BBB_RESET_3V3: track 219.3 -> 220.7 mm
- net SERVO_RUDDER_3V3: track 180.3 -> 179.2 mm
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