File: hardware/electronics/ControlBoard/Hackerboat Control Board.sch (EAGLE design)
At the start: 287 parts, among them IC1 74AHC1G08DBV, IC2 74AUC1G06DBV, IC3 74AHC1G04DBV, IC4 V7805, IC5 7805TV, T1 AO4407A, U1 IPS6041G, U10 INA169, U11 IPS6041G, U12 INA169, U15 TPS54331, U18 ADC128D818, U19 ADC128D818, U2 IPS6041G, U20 IPS6041G, U21 INA169, U22 IPS6041G, U23 INA169, U24 IPS6041G, U25 INA169, U27 INA169, U29 TPS61175, U3 INA169, U4 IPS6041G, U5 INA169, U6 IPS6041G, U7 INA169, U8 IPS6041G, U9 INA169

Commit message: More fiddling around with the silkscreen
Parts:
- renumbered J4 to ENABLE/DISARM, U$6 to U28
Changed lines of the file:
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@@
 <part name="J2" library="SparkFun-Connectors" deviceset="M03" device="LOCK"/>
 <part name="J3" library="SparkFun-Connectors" deviceset="M04" device="LOCK"/>
-<part name="J4" library="SparkFun-Connectors" deviceset="M05" device="LOCK"/>
+<part name="ENABLE/DISARM" library="SparkFun-Connectors" deviceset="M05" device="LOCK"/>
 <part name="J5" library="SparkFun-Connectors" deviceset="M09" device="LOCK"/>
 <part name="J6" library="SparkFun-Connectors" deviceset="M10" device="LOCK"/>
@@
 <part name="GND102" library="supply1" deviceset="GND" device=""/>
 <part name="AUX_GPIO" library="SparkFun-Connectors" deviceset="M06X2" device="PTH_FEMALE" value="2X6 FEMALE"/>
-<part name="U$6" library="SparkFun-DigitalIC" deviceset="RS485" device="SOIC"/>
+<part name="U28" library="SparkFun-DigitalIC" deviceset="RS485" device="SOIC"/>
 <part name="RS485" library="con-molex-c-grid-sl" deviceset="HEADER_POS3_?" device="70555"/>
 <part name="J11" library="SparkFun-Connectors" deviceset="M03" device="LOCK"/>
@@
 </instance>
 <instance part="GND47" gate="1" x="88.9" y="5.08" rot="MR0"/>
-<instance part="J4" gate="G$1" x="165.1" y="33.02" rot="R180"/>
+<instance part="ENABLE/DISARM" gate="G$1" x="165.1" y="33.02" rot="R180"/>
 <instance part="RLY0" gate="G$1" x="182.88" y="160.02"/>
 <instance part="R62" gate="G$1" x="182.88" y="167.64" rot="R90"/>
@@
 <wire x1="88.9" y1="10.16" x2="88.9" y2="7.62" width="0.1524" layer="91"/>
 <wire x1="157.48" y1="33.02" x2="142.24" y2="33.02" width="0.1524" layer="91"/>
-<pinref part="J4" gate="G$1" pin="3"/>
+<pinref part="ENABLE/DISARM" gate="G$1" pin="3"/>
 <pinref part="ENABLE" gate="G$1" pin="C"/>
 <wire x1="78.74" y1="10.16" x2="88.9" y2="10.16" width="0.1524" layer="91"/>
@@
 <wire x1="53.34" y1="30.48" x2="45.72" y2="30.48" width="0.1524" layer="91"/>
 <wire x1="157.48" y1="30.48" x2="142.24" y2="30.48" width="0.1524" layer="91"/>
-<pinref part="J4" gate="G$1" pin="4"/>
+<pinref part="ENABLE/DISARM" gate="G$1" pin="4"/>
 <pinref part="R68" gate="G$1" pin="2"/>
 <wire x1="55.88" y1="20.32" x2="53.34" y2="20.32" width="0.1524" layer="91"/>
@@
 <segment>
 <pinref part="POWER_STATE" gate="G$1" pin="1"/>
-<pinref part="J4" gate="G$1" pin="1"/>
+<pinref part="ENABLE/DISARM" gate="G$1" pin="1"/>
 <wire x1="157.48" y1="38.1" x2="142.24" y2="38.1" width="0.1524" layer="91"/>
 <pinref part="R89" gate="G$1" pin="1"/>
@@
 <segment>
 <pinref part="POWER_STATE" gate="G$1" pin="2"/>
-<pinref part="J4" gate="G$1" pin="2"/>
+<pinref part="ENABLE/DISARM" gate="G$1" pin="2"/>
 <wire x1="157.48" y1="35.56" x2="142.24" y2="35.56" width="0.1524" layer="91"/>
 <pinref part="R90" gate="G$1" pin="1"/>
@@
 <segment>
 <pinref part="POWER_STATE" gate="G$1" pin="5"/>
-<pinref part="J4" gate="G$1" pin="5"/>
+<pinref part="ENABLE/DISARM" gate="G$1" pin="5"/>
 <wire x1="157.48" y1="27.94" x2="142.24" y2="27.94" width="0.1524" layer="91"/>
 <wire x1="142.24" y1="27.94" x2="134.62" y2="27.94" width="0.1524" layer="91"/>
@@
 <instance part="C9" gate="G$1" x="111.76" y="147.32"/>
 <instance part="C10" gate="G$1" x="114.3" y="88.9"/>
-<instance part="U$6" gate="G$1" x="78.74" y="22.86"/>
+<instance part="U28" gate="G$1" x="78.74" y="22.86"/>
 <instance part="RS485" gate="G$1" x="134.62" y="20.32"/>
 <instance part="J11" gate="J$1" x="137.16" y="35.56" rot="R180"/>
@@
 </segment>
 <segment>
-<pinref part="U$6" gate="G$1" pin="GND"/>
+<pinref part="U28" gate="G$1" pin="GND"/>
 <pinref part="RS485" gate="G$1" pin="3"/>
 <wire x1="129.54" y1="17.78" x2="127" y2="17.78" width="0.1524" layer="91"/>
@@
 </segment>
 <segment>
-<pinref part="U$6" gate="G$1" pin="VCC"/>
+<pinref part="U28" gate="G$1" pin="VCC"/>
 <wire x1="93.98" y1="25.4" x2="99.06" y2="25.4" width="0.1524" layer="91"/>
 <wire x1="99.06" y1="25.4" x2="99.06" y2="27.94" width="0.1524" layer="91"/>
@@
 <net name="N$27" class="0">
 <segment>
-<pinref part="U$6" gate="G$1" pin="B"/>
+<pinref part="U28" gate="G$1" pin="B"/>
 <pinref part="RS485" gate="G$1" pin="1"/>
 <wire x1="129.54" y1="22.86" x2="121.92" y2="22.86" width="0.1524" layer="91"/>
@@
 <net name="N$86" class="0">
 <segment>
-<pinref part="U$6" gate="G$1" pin="A"/>
+<pinref part="U28" gate="G$1" pin="A"/>
 <pinref part="RS485" gate="G$1" pin="2"/>
 <wire x1="129.54" y1="20.32" x2="124.46" y2="20.32" width="0.1524" layer="91"/>
@@
 <net name="RS_485_DIR_SELECT_5V" class="0">
 <segment>
-<pinref part="U$6" gate="G$1" pin="/RE"/>
+<pinref part="U28" gate="G$1" pin="/RE"/>
 <wire x1="68.58" y1="22.86" x2="66.04" y2="22.86" width="0.1524" layer="91"/>
-<pinref part="U$6" gate="G$1" pin="DE"/>
+<pinref part="U28" gate="G$1" pin="DE"/>
 <wire x1="66.04" y1="22.86" x2="63.5" y2="22.86" width="0.1524" layer="91"/>
 <wire x1="68.58" y1="20.32" x2="66.04" y2="20.32" width="0.1524" layer="91"/>
@@
 <net name="BBB_UART1_TX_5V" class="0">
 <segment>
-<pinref part="U$6" gate="G$1" pin="DI"/>
+<pinref part="U28" gate="G$1" pin="DI"/>
 <wire x1="68.58" y1="17.78" x2="63.5" y2="17.78" width="0.1524" layer="91"/>
 <label x="63.5" y="17.78" size="1.778" layer="95" rot="R180" xref="yes"/>
@@
 <net name="BBB_UART1_RX_5V" class="0">
 <segment>
-<pinref part="U$6" gate="G$1" pin="RO"/>
+<pinref part="U28" gate="G$1" pin="RO"/>
 <wire x1="68.58" y1="25.4" x2="66.04" y2="25.4" width="0.1524" layer="91"/>
 <wire x1="66.04" y1="25.4" x2="66.04" y2="27.94" width="0.1524" layer="91"/>

Commit message: A bit of BoM and silkscreen cleanup
Parts:
- 15V-ENB, J1, J10, J11, J2, J9: BOM (none) -> EXCLUDE
- 5V-STAT, 7V4-STAT, ACC_POWER, AUX_GPIO, BBB_CONSOLE, BBB_RESET, BLOWN, C18, C20, C26, C27, C30, C31, C33, C34, C41, C42, C43, C44, C45, C46, C49, C50, CELL, D1, D10, D11, D12, D13, D14, D15, D16, D17, D18, D19, D2, D20, D21, D22, D23, D24, D25, D26, D27, D28, D3, D36, D4, D5, D6, D7, D8, D9, DISARM, ENABLE, ENABLE/DISARM, F2, FAULT_0, FAULT_1, FAULT_2, FAULT_3, FAULT_4, FAULT_5, FAULT_DISARM, FAULT_ENABLE, FAULT_HORN, GPS, HORN, HORN-RLY, IC1, IC2, IC3, IMU, J3, J5, J6, J7, L2, L3, MOTOR-CTRL-RELAYS, POE-DEVICE, POE-LAN, POWER_INPUT, POWER_MON, POWER_STATE, PWR, R10, R11, R110, R111, R112, R113, R12, R16, R17, R18, R19, R20, R26, R27, R28, R31, R32, R33, R37, R4, R40, R41, R45, R46, R47, R49, R5, R50, R51, R52, R53, R54, R55, R56, R58, R59, R6, R60, R61, R72, R73, R74, R78, R79, R80, R84, R85, R86, REV, RLY0, RLY1, RLY2, RLY3, RLY4, RLY5, RS485, SBUS-IN, SBUS-OUT, SERIAL_CONSOLE, SJ2, STATUS_LIGHTS, STEERING, U$2, U$3, U$4, U$5, U1, U10, U11, U12, U13, U15, U16, U17, U18, U19, U2, U20, U21, U22, U23, U24, U25, U26, U27, U28, U29, U3, U4, U5, U6, U7, U8, U9: PARTNO (none) -> *
- C1, C10, C11, C12, C13, C14, C15, C16, C2, C3, C32, C35, C36, C37, C38, C39, C4, C40, C47, C48, C5, C6, C7, C8, C9: PARTNO (none) -> CC0603KRX7R9BB104
- C17, C19, C28, C29: PARTNO (none) -> UMK325BJ106MM
- R1, R13, R14, R15, R2, R25, R29, R3, R30, R34, R35, R36, R42, R43, R44, R48, R57, R69, R7, R70, R71, R75, R76, R77, R8, R81, R82, R83, R9, R97, R98, R99: PARTNO (none) -> RNCP0603FTD10K0
- R100, R101, R102, R103, R104, R105, R106, R107, R108, R109, R24, R38, R39, R62, R63, R64, R65, R66, R67, R68, R87, R88, R89, R90, R91, R92, R93, R94, R95, R96: PARTNO (none) -> RMCF0603FT1K00
