File: hardware/electronics/ControlBoard/HackerboatControlBoard.brd (EAGLE design)
At the start: 114.3 x 195.6 mm, 287 parts, among them IC1 74AHC1G08DBV, IC2 74AUC1G06DBV, IC3 74AHC1G04DBV, IC4 V7805, IC5 7805TV, T1 AO4407A, U1 IPS6041G, U10 INA169, U11 IPS6041G, U12 INA169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

Commit message: Control board BoM complete
Parts:
- C33: value 7u5 -> 7p5
- C41, C42, C49, C50: value 1000p -> 22n
- IC4: value V7805 -> V7805-2000
- IC5: value 7805TV -> V7805-2000
- R110, R111, R112, R113: value (none) -> 10K
