File: hardware/electronics/PowerDistribution/PowerDistributionBoard.brd (EAGLE design)
At the start: 122.6 x 50.8 mm, 82 parts, among them IC1 LM556D, IC2 74AHC1G02DBV, IC3 74AHC1G02DBV, K1 EC2-12TNU, U1 IPS6041G, U2 IPS6041G, U3 V_REG_317SMD

Commit message: Fixed some issues with .gitignore and added some values and attributes to the power distribution board
Parts:
- C10, C2, C9: value (none) -> 10u
- C4: value (none) -> 2u2
- C5, C6: value (none) -> 1u
- C7, C8: value (none) -> 100n
- R1, R2: value (none) -> 470K
- R10, R11, R12, R13, R14, R15, R16, R17, R18, R19, R20, R21, R22, R7, R8, R9: value (none) -> 1K
- R3: value (none) -> 1M
- R4, R5, R6: value (none) -> 10K
